File: PCB_DES/LOCK_EDGE_BASEBOARD/LOCK_EDGE_BASEBOARD.kicad_pcb (KiCad board)
At the start: 2 copper layers, 100 x 100 mm, 5 parts, among them J1 Servo_Motor_3Pin, J2 Arduino_Header, U2 RFID-RC522, U3 ESP32-C5-DevKit-V2

Commit message: Update
Parts:
- added J3: INA228_Breakout, Library:INA228_Breakout_Socket, F.Cu at (136.7, 85.8)
Connections:
- J2 pad 10: /RFID_IRQ -> /RFID_RST
- J2 pad 12: /TOUCH_CS -> /RFID_IRQ
- J2 pad 16: /RFID_RST -> /INA_ALRT
- J2 pad 17: /TFT_CS -> /TOUCH_IRQ
- J2 pad 18: /TFT_RESET -> /TOUCH_CS
- J2 pad 21: /TOUCH_IRQ -> /TFT_RESET
- J2 pad 24: /TFT_LED -> /TFT_CS
- J2 pad 30: unconnected-(J2-SDA-Pad30) -> /INA_SDA
- J2 pad 31: unconnected-(J2-SCL-Pad31) -> /INA_SCL
- U1 pad 7: /TFT_LED -> VDD_3V3
Routing:
- net VDD_3V3: track 40.5 -> 217.3 mm
- net /INA_SCL: track 0.00 -> 69.7 mm, vias 0 -> 1
- net /TFT_LED: track 67.4 -> 0.00 mm
- net /INA_SDA: track 0.00 -> 64.5 mm, vias 0 -> 1
- net VDD_5V0: track 181.8 -> 241.2 mm
- net /TOUCH_IRQ: track 47.9 -> 95.9 mm
- net /TFT_CS: track 98.8 -> 53.0 mm
- net /TFT_RESET: track 89.8 -> 55.8 mm
- net /TOUCH_CS: track 113.8 -> 88.7 mm
- net /SPI_MOSI: track 231.8 -> 254.0 mm
- net /SPI_MISO: track 242.4 -> 261.4 mm
- net /INA_ALRT: track 0.00 -> 18.6 mm
- net /RFID_RST: track 75.9 -> 57.6 mm
- net /TFT_DC: track 81.0 -> 66.8 mm
- net /RFID_IRQ: track 66.0 -> 64.1 mm
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
Commit message: Update
Parts:
- added JP1: JP_BOOT1, Library:JP_Header_1x03_P2.54mm, F.Cu at (94.8, 85.8)
- added R1: 1K, Resistor_SMD:R_1206_3216Metric_Pad1.30x1.75mm_HandSolder, F.Cu at (88.9, 90.0)
- added SW1: SW_Push, Library:SW_PUSH_6mm, F.Cu at (91.8, 90.0)
Connections:
- J2 pad 25: /SPI_MISO -> /SPI_MOSI
- J2 pad 26: /SPI_MOSI -> /SPI_MISO
Routing:
- net VDD_3V3: track 217.3 -> 229.3 mm
- net Net-(R1-Pad1): track 0.00 -> 11.5 mm
- net /BOOT1_SIM: track 0.00 -> 11.1 mm
- net /SPI_MOSI: track 254.0 -> 257.3 mm
- net VDDIO: track 0.00 -> 3.08 mm
- net /SPI_MISO: track 261.4 -> 263.6 mm, vias 0 -> 2
- net GND: vias 170 -> 465
Other:
- board text added: "{ "ViaStitching": "0.2", "stitch_zone_0": { "HSpacing": "3", "VSpacing": "3", "HOffset": "0", "VOffset": "0", "Clearance": "0.25", "Randomize": false } }"
