File: PCB_DES/LOCK_EDGE_BASEBOARD/LOCK_EDGE_BASEBOARD.kicad_sch (KiCad schematic)
At the start: 0 parts

Commit message: Update
Parts:
- added J1: Servo_Motor_3Pin, Library:Servo_Header_1x03_P2.54mm, symbol servo-motor-3pin:Servo_Motor_3Pin
- added J2: Arduino_Header, Library:Arduino_Header, symbol arduino-header:Arduino_Header
- added U1: (no value), Library:TFT_240x320_SPI_Touch_14Pin, symbol tft-240x320-spi:TFT_240x320_SPI_Touch_14P
- added U2: RFID-RC522, Library:RFID-RC522_Header_1x08_P2.54mm, symbol rfid-rc522:RFID-RC522
- added U3: ESP32-C5-DevKit-V2, Library:ESP32-C5-DevKit-V2, symbol esp32-c5-devkit-v2:ESP32-C5-DevKit-V2

Commit message: update
Connections:
- net SERVO_PWM: now reaches J1.1 (SIG)
- net SERVO_PWM: now also J2.23 (D9)
- net VDD_5V0: now reaches J1.2 (VCC)
- net VDD_5V0: now also J2.3 (5V), U1.14 (VCC), U3.17 (5V)
- net GND: now reaches J1.3 (GND)
- net GND: now also J2.28 (GND), J2.5 (GND), J2.6 (GND), U1.13 (GND), U2.6 (GND), U3.1 (GND), U3.12 (GND), U3.15 (GND), U3.16 (GND)
- net RFID_IRQ: now reaches J2.10 (A2)
- net RFID_IRQ: now also U2.5 (IRQ)
- net SD_CS: now reaches J2.11 (A3)
- net SD_CS: now also U1.15 (SD_CS)
- net TOUCH_CS: now reaches J2.12 (A4)
- net TOUCH_CS: now also U1.4 (T_CS)
- net ESP32_CS: now reaches J2.13 (A5)
- net ESP32_CS: now also U3.21 (GPIO9)
- net RFID_RST: now reaches J2.16 (D2)
- net RFID_RST: now also U2.7 (RST)
- net TFT_CS: now reaches J2.17 (D3)
- net TFT_CS: now also U1.12 (CS)
- net TFT_RESET: now reaches J2.18 (D4)
- net TFT_RESET: now also U1.11 (RESET)
- net TFT_DC: now reaches J2.19 (D5)
- net TFT_DC: now also U1.10 (DC)
- net TOUCH_IRQ: now reaches J2.21 (D7)
- net TOUCH_IRQ: now also U1.1 (T_IRQ)
- net RFID_CS: now reaches J2.22 (D8)
- net RFID_CS: now also U2.1 (SS)
- net TFT_LED: now reaches J2.24 (D10)
- net TFT_LED: now also U1.7 (LED)
- net SPI_MISO: now reaches J2.25 (D11)
- net SPI_MISO: now also U1.17 (SD_MISO), U1.2 (T_DO), U1.6 (MISO), U2.4 (MISO), U3.22 (GPIO8)
- net SPI_MOSI: now reaches J2.26 (D12)
- net SPI_MOSI: now also U1.16 (SD_MOSI), U1.3 (T_DIN), U1.9 (MOSI), U2.3 (MOSI), U3.20 (GPIO10)
- net SPI_SCK: now reaches J2.27 (D13)
- net SPI_SCK: now also U1.18 (SD_SCK), U1.5 (T_CLK), U1.8 (SCK), U2.2 (SCK), U3.24 (GPIO6)
- net VDD_3V3: now reaches J2.4 (3.3V)
- net VDD_3V3: now also U2.8 (3.3V)
- no-connect marks 0 -> 33
Other:
- moved on the sheet: J1, U2, U3

Commit message: Update
Parts:
- added J3: INA228_Breakout, Library:INA228_Breakout_Socket, symbol ina228-breakout:INA228_Breakout
Connections:
- net GND: now also J3.2 (GND)
- net RFID_IRQ: now also J2.12 (A4); no longer J2.10 (A2)
- net RFID_RST: now also J2.10 (A2); no longer J2.16 (D2)
- net TFT_CS: now also J2.24 (D10); no longer J2.17 (D3)
- net TFT_RESET: now also J2.21 (D7); no longer J2.18 (D4)
- net TOUCH_CS: now also J2.18 (D4); no longer J2.12 (A4)
- net TOUCH_IRQ: now also J2.17 (D3); no longer J2.21 (D7)
- net VDD_3V3: now also U1.7 (LED), J3.1 (VCC)
- net INA_SDA: now reaches J2.30 (SDA)
- net INA_SDA: now also J3.4 (SDA)
- net INA_SCL: now reaches J2.31 (SCL)
- net INA_SCL: now also J3.3 (SCL)
- removed net TFT_LED: J2.24 (D10), U1.7 (LED)
- new net INA_ALRT: J2.16 (D2), J3.8 (ALRT)
- no-connect marks 33 -> 34

Commit message: Update
Parts:
- added JP1: JP_BOOT1, Library:JP_Header_1x03_P2.54mm, symbol Connector_Generic:Conn_01x03
- added R1: 1K, Resistor_SMD:R_1206_3216Metric_Pad1.30x1.75mm_HandSolder, symbol Device:R
- added SW1: SW_Push, Library:SW_PUSH_6mm, symbol Switch:SW_Push
Connections:
- net GND: now also JP1.1 (Pin_1)
- net SPI_MISO: now also J2.26 (D12); no longer J2.25 (D11)
- net SPI_MOSI: now also J2.25 (D11); no longer J2.26 (D12)
- new net: R1.1, SW1.2
- new net BOOT1_SIM: JP1.2 (Pin_2), SW1.1
- new net VDDIO: JP1.3 (Pin_3), R1.2
